File: sch/thinkpad_keyboard_usb.kicad_pcb (KiCad board)
At the start: 2 copper layers, 45 x 110 mm, 44 parts, among them IC1 MCP1603T-330IOT, J1 Conn_02x20_Odd_Even_MountingP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, J2 UART, J3 SWD, J4 USB_C_Receptacle_USB2.0, U1 USBLC6-2SC6, U2 STM32H503RBTx

Commit message: Added board name and version to silk
Other:
- board text added: "ThinkPad keyboard to USB ${REVISION}"
- board text added: "https://nathandumont.com/blog/usb-thinkpad-keyboard"
